File: Learning_Activities/slike/RobDuino_Basics_Electronics.kicad_sch (KiCad schematic)
At the start: 14 parts, among them M1 Motor_DC_ALT, SW1 SW_Push, SW4 SW_Push, SW5 SW_Push

Commit message: nekaj posodobitev
Other:
- added sheet A (untitled.kicad_sch)
- moved on the sheet: A1, BT1, L1, LED1, LED2, M1, R1, R2, R3, R4, R6, SW1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
